Commit message: Update diff_wheeled_robot.urdf.xacro

File: workshop_robot/mastering_ros_robot_description_pkg (copy)/urdf/diff_wheeled_robot.urdf.xacro (robot description, xacro)
@@ -56,5 +56,5 @@
       <origin rpy="0 0 0" xyz="0 0 0"/>
       <geometry>
-        <box size="0.2 0.3 0.01"/>
+         <box size="0.33 0.3 0.03"/>
       </geometry>
       <material name="Red"/>
@@ -63,5 +63,5 @@
       <origin rpy="0 0 0 " xyz="0 0 0"/>
       <geometry>
-        <box size="0.2 0.3 0.01"/>
+         <box size="0.33 0.3 0.03"/>
 </geometry>
     </collision>
